Commit message: Changing the camera angle of the Husky from 0* to 15* up wards (~=-0.25 rad)

File: src/forest_guard_sim/urdf/husky.urdf.xacro (robot description, xacro)
@@ -121,5 +121,5 @@
   </link>
   <joint name="camera_joint" type="fixed">
-    <origin xyz="0.45 0.0 0.25" rpy="0 0 0"/> <!-- 0.5 0.0 0.9 -->
+    <origin xyz="0.45 0.0 0.25" rpy="0 -0.25 0"/> <!-- 0.5 0.0 0.9 -->
     <parent link="base_link"/>
     <child link="camera_link"/>

Commit message: Large Reversion

File: src/forest_guard_sim/urdf/husky.urdf.xacro (robot description, xacro)
@@ -121,5 +121,5 @@
   </link>
   <joint name="camera_joint" type="fixed">
-    <origin xyz="0.45 0.0 0.25" rpy="0 -0.25 0"/> <!-- 0.5 0.0 0.9 -->
+    <origin xyz="0.45 0.0 0.25" rpy="0 0 0"/> <!-- 0.5 0.0 0.9 -->
     <parent link="base_link"/>
     <child link="camera_link"/>
