Commit message: Renamed everything named john to forestguard_sim

File: src/forestguard_sim/urdf/husky.gazebo.xacro (robot description, xacro)
@@ -4,5 +4,5 @@
   <xacro:arg name="camera_visual" default="false"/>
   <xacro:arg name="imu_visual"    default="false"/>
-  <xacro:include filename="$(find john)/urdf/wheel.urdf.xacro"/>
+  <xacro:include filename="$(find forestguard_sim)/urdf/wheel.urdf.xacro"/>
   <gazebo reference="imu_link">
     <sensor type="imu" name="imu">

File: src/forestguard_sim/urdf/husky.urdf.xacro (robot description, xacro)
@@ -1,7 +1,7 @@
 <?xml version="1.0" ?>
 <robot name="husky" xmlns:xacro="http://ros.org/wiki/xacro">
-  <xacro:include filename="$(find john)/urdf/common_properties.urdf.xacro"/>
-  <xacro:include filename="$(find john)/urdf/husky.gazebo.xacro"/>
-  <xacro:include filename="$(find john)/urdf/wheel.urdf.xacro"/>
+  <xacro:include filename="$(find forestguard_sim)/urdf/common_properties.urdf.xacro"/>
+  <xacro:include filename="$(find forestguard_sim)/urdf/husky.gazebo.xacro"/>
+  <xacro:include filename="$(find forestguard_sim)/urdf/wheel.urdf.xacro"/>
   <xacro:property name="r200_cam_rgb_px" value="0.005"/>
   <xacro:property name="r200_cam_rgb_py" value="0.018"/>
@@ -12,5 +12,5 @@
       <origin xyz="0 0 0.0" rpy="0 0 0"/>
       <geometry>
-        <mesh filename="file://$(find john)/urdf/meshes/base_link.dae"/>
+        <mesh filename="file://$(find forestguard_sim)/urdf/meshes/base_link.dae"/>
       </geometry>
       <material name="black"/>
@@ -19,5 +19,5 @@
       <origin xyz="0.48 0 0.091" rpy="0 0 0"/>
       <geometry>
-        <mesh filename="file://$(find john)/urdf/meshes/bumper.dae"/>
+        <mesh filename="file://$(find forestguard_sim)/urdf/meshes/bumper.dae"/>
       </geometry>
       <material name="black"/>
@@ -26,5 +26,5 @@
       <origin xyz="-0.48 0 0.091" rpy="0 0 3.14159"/>
       <geometry>
-        <mesh filename="file://$(find john)/urdf/meshes/bumper.dae"/>
+        <mesh filename="file://$(find forestguard_sim)/urdf/meshes/bumper.dae"/>
       </geometry>
       <material name="black"/>
@@ -33,5 +33,5 @@
       <origin xyz="0 0 0" rpy="0 0 0"/>
       <geometry>
-        <mesh filename="file://$(find john)/urdf/meshes/top_chassis.dae"/>
+        <mesh filename="file://$(find forestguard_sim)/urdf/meshes/top_chassis.dae"/>
       </geometry>
     </visual>
@@ -39,5 +39,5 @@
       <origin xyz="0.0812 0 0.245" rpy="0 0 0"/>
       <geometry>
-        <mesh filename="file://$(find john)/urdf/meshes/top_plate.dae"/>
+        <mesh filename="file://$(find forestguard_sim)/urdf/meshes/top_plate.dae"/>
       </geometry>
       <material name="black"/>
@@ -46,5 +46,5 @@
       <origin xyz="0.0012 0 0.251" rpy="0 0 0"/>
       <geometry>
-        <mesh filename="file://$(find john)/urdf/meshes/jpl04_arch_nosensor.stl"/>
+        <mesh filename="file://$(find forestguard_sim)/urdf/meshes/jpl04_arch_nosensor.stl"/>
       </geometry>
       <material name="black"/>
@@ -71,5 +71,5 @@
       <origin xyz="0.0812 0 0.245" rpy="0 0 0"/>
       <geometry>
-        <mesh filename="file://$(find john)/urdf/meshes/top_plate.dae"/>
+        <mesh filename="file://$(find forestguard_sim)/urdf/meshes/top_plate.dae"/>
       </geometry>
     </collision>

File: src/forestguard_sim/urdf/wheel.urdf.xacro (robot description, xacro)
@@ -9,5 +9,5 @@
         <origin xyz="0 0 0" rpy="0 0 0"/>
         <geometry>
-          <mesh filename="file://$(find john)/urdf/meshes/wheel.dae"/>
+          <mesh filename="file://$(find forestguard_sim)/urdf/meshes/wheel.dae"/>
         </geometry>
       </visual>

Commit message: Final Push for Handover

File: src/forestguard_sim/urdf/husky.gazebo.xacro (robot description, xacro)
@@ -170,3 +170,87 @@
     </sensor>
   </gazebo>
+  <!-- Rear-facing RGBD camera -->
+  <gazebo reference="rear_camera_link">
+    <sensor name="rear_rgbd_camera" type="rgbd_camera">
+      <pose>0 0 0 0 0 0</pose>
+      <camera>
+        <horizontal_fov>2.0944</horizontal_fov>
+        <image>
+          <width>720</width>
+          <height>480</height>
+        </image>
+        <clip>
+          <near>0.1</near>
+          <far>40</far>
+        </clip>
+        <depth_camera>
+          <clip>
+            <near>0.4</near>
+            <far>10</far>
+          </clip>
+        </depth_camera>
+      </camera>
+      <always_on>1</always_on>
+      <update_rate>3</update_rate>
+      <visualize>$(arg camera_visual)</visualize>
+      <topic>/model/husky/rear_camera</topic>
+      <gz_frame_id>rear_camera_link</gz_frame_id>
+    </sensor>
+  </gazebo>
+  <!-- Left-facing RGBD camera -->
+  <gazebo reference="left_camera_link">
+    <sensor name="left_rgbd_camera" type="rgbd_camera">
+      <pose>0 0 0 0 0 0</pose>
+      <camera>
+        <horizontal_fov>2.0944</horizontal_fov>
+        <image>
+          <width>720</width>
+          <height>480</height>
+        </image>
+        <clip>
+          <near>0.1</near>
+          <far>40</far>
+        </clip>
+        <depth_camera>
+          <clip>
+            <near>0.4</near>
+            <far>10</far>
+          </clip>
+        </depth_camera>
+      </camera>
+      <always_on>1</always_on>
+      <update_rate>3</update_rate>
+      <visualize>$(arg camera_visual)</visualize>
+      <topic>/model/husky/left_camera</topic>
+      <gz_frame_id>left_camera_link</gz_frame_id>
+    </sensor>
+  </gazebo>
+  <!-- Right-facing RGBD camera -->
+  <gazebo reference="right_camera_link">
+    <sensor name="right_rgbd_camera" type="rgbd_camera">
+      <pose>0 0 0 0 0 0</pose>
+      <camera>
+        <horizontal_fov>2.0944</horizontal_fov>
+        <image>
+          <width>720</width>
+          <height>480</height>
+        </image>
+        <clip>
+          <near>0.1</near>
+          <far>40</far>
+        </clip>
+        <depth_camera>
+          <clip>
+            <near>0.4</near>
+            <far>10</far>
+          </clip>
+        </depth_camera>
+      </camera>
+      <always_on>1</always_on>
+      <update_rate>3</update_rate>
+      <visualize>$(arg camera_visual)</visualize>
+      <topic>/model/husky/right_camera</topic>
+      <gz_frame_id>right_camera_link</gz_frame_id>
+    </sensor>
+  </gazebo>
 </robot>

File: src/forestguard_sim/urdf/husky.urdf.xacro (robot description, xacro)
@@ -165,3 +165,141 @@
   </joint>
   <link name="camera_depth_optical_frame"/>
+  <!-- Rear camera assembly -->
+  <joint name="rear_camera_joint" type="fixed">
+    <origin xyz="-0.285 0.0 0.275" rpy="0 0.250 3.14159"/>
+    <parent link="base_link"/>
+    <child link="rear_camera_link"/>
+  </joint>
+  <link name="rear_camera_link">
+    <visual>
+      <origin xyz="0 0 0" rpy="0 0 0"/>
+      <geometry>
+        <box size="0.02 0.08 0.05"/>
+      </geometry>
+      <material name="dark"/>
+    </visual>
+    <visual>
+      <origin xyz="0.01 0 0" rpy="0 1.57 3.14159"/>
+      <geometry>
+        <cylinder length="0.03" radius="0.02"/>
+      </geometry>
+      <material name="dark"/>
+    </visual>
+  </link>
+  <joint name="rear_camera_rgb_joint" type="fixed">
+    <origin xyz="${r200_cam_rgb_px} ${r200_cam_rgb_py} ${r200_cam_rgb_pz}" rpy="0 0 0"/>
+    <parent link="rear_camera_link"/>
+    <child link="rear_camera_rgb_frame"/>
+  </joint>
+  <link name="rear_camera_rgb_frame"/>
+  <joint name="rear_camera_rgb_optical_joint" type="fixed">
+    <origin xyz="0 0 0" rpy="-1.57 0 -1.57"/>
+    <parent link="rear_camera_rgb_frame"/>
+    <child link="rear_camera_rgb_optical_frame"/>
+  </joint>
+  <link name="rear_camera_rgb_optical_frame"/>
+  <joint name="rear_camera_depth_joint" type="fixed">
+    <origin xyz="${r200_cam_rgb_px} ${r200_cam_rgb_py + r200_cam_depth_offset} ${r200_cam_rgb_pz}" rpy="0 0 0"/>
+    <parent link="rear_camera_link"/>
+    <child link="rear_camera_depth_frame"/>
+  </joint>
+  <link name="rear_camera_depth_frame"/>
+  <joint name="rear_camera_depth_optical_joint" type="fixed">
+    <origin xyz="0 0 0" rpy="-1.57 0 -1.57"/>
+    <parent link="rear_camera_depth_frame"/>
+    <child link="rear_camera_depth_optical_frame"/>
+  </joint>
+  <link name="rear_camera_depth_optical_frame"/>
+  <!-- Left roll-cage camera -->
+  <joint name="left_camera_joint" type="fixed">
+    <origin xyz="0.0 0.24 0.58" rpy="0 0.5 1.5708"/>
+    <parent link="base_link"/>
+    <child link="left_camera_link"/>
+  </joint>
+  <link name="left_camera_link">
+    <visual>
+      <origin xyz="0 0 0" rpy="0 0 0"/>
+      <geometry>
+        <box size="0.02 0.08 0.05"/>
+      </geometry>
+      <material name="dark"/>
+    </visual>
+    <visual>
+      <origin xyz="0.02 0 0" rpy="0 1.57 0"/>
+      <geometry>
+        <cylinder length="0.03" radius="0.02"/>
+      </geometry>
+      <material name="dark"/>
+    </visual>
+  </link>
+  <joint name="left_camera_rgb_joint" type="fixed">
+    <origin xyz="${r200_cam_rgb_px} ${r200_cam_rgb_py} ${r200_cam_rgb_pz}" rpy="0 0 0"/>
+    <parent link="left_camera_link"/>
+    <child link="left_camera_rgb_frame"/>
+  </joint>
+  <link name="left_camera_rgb_frame"/>
+  <joint name="left_camera_rgb_optical_joint" type="fixed">
+    <origin xyz="0 0 0" rpy="-1.57 0 -1.57"/>
+    <parent link="left_camera_rgb_frame"/>
+    <child link="left_camera_rgb_optical_frame"/>
+  </joint>
+  <link name="left_camera_rgb_optical_frame"/>
+  <joint name="left_camera_depth_joint" type="fixed">
+    <origin xyz="${r200_cam_rgb_px} ${r200_cam_rgb_py + r200_cam_depth_offset} ${r200_cam_rgb_pz}" rpy="0 0 0"/>
+    <parent link="left_camera_link"/>
+    <child link="left_camera_depth_frame"/>
+  </joint>
+  <link name="left_camera_depth_frame"/>
+  <joint name="left_camera_depth_optical_joint" type="fixed">
+    <origin xyz="0 0 0" rpy="-1.57 0 -1.57"/>
+    <parent link="left_camera_depth_frame"/>
+    <child link="left_camera_depth_optical_frame"/>
+  </joint>
+  <link name="left_camera_depth_optical_frame"/>
+  <!-- Right roll-cage camera -->
+  <joint name="right_camera_joint" type="fixed">
+    <origin xyz="0.0 -0.24 0.58" rpy="0 0.5 -1.5708"/>
+    <parent link="base_link"/>
+    <child link="right_camera_link"/>
+  </joint>
+  <link name="right_camera_link">
+    <visual>
+      <origin xyz="0 0 0" rpy="0 0 0"/>
+      <geometry>
+        <box size="0.02 0.08 0.05"/>
+      </geometry>
+      <material name="dark"/>
+    </visual>
+    <visual>
+      <origin xyz="0.02 0 0" rpy="0 1.57 0"/>
+      <geometry>
+        <cylinder length="0.03" radius="0.02"/>
+      </geometry>
+      <material name="dark"/>
+    </visual>
+  </link>
+  <joint name="right_camera_rgb_joint" type="fixed">
+    <origin xyz="${r200_cam_rgb_px} ${r200_cam_rgb_py} ${r200_cam_rgb_pz}" rpy="0 0 0"/>
+    <parent link="right_camera_link"/>
+    <child link="right_camera_rgb_frame"/>
+  </joint>
+  <link name="right_camera_rgb_frame"/>
+  <joint name="right_camera_rgb_optical_joint" type="fixed">
+    <origin xyz="0 0 0" rpy="-1.57 0 -1.57"/>
+    <parent link="right_camera_rgb_frame"/>
+    <child link="right_camera_rgb_optical_frame"/>
+  </joint>
+  <link name="right_camera_rgb_optical_frame"/>
+  <joint name="right_camera_depth_joint" type="fixed">
+    <origin xyz="${r200_cam_rgb_px} ${r200_cam_rgb_py + r200_cam_depth_offset} ${r200_cam_rgb_pz}" rpy="0 0 0"/>
+    <parent link="right_camera_link"/>
+    <child link="right_camera_depth_frame"/>
+  </joint>
+  <link name="right_camera_depth_frame"/>
+  <joint name="right_camera_depth_optical_joint" type="fixed">
+    <origin xyz="0 0 0" rpy="-1.57 0 -1.57"/>
+    <parent link="right_camera_depth_frame"/>
+    <child link="right_camera_depth_optical_frame"/>
+  </joint>
+  <link name="right_camera_depth_optical_frame"/>
 </robot>
